File: Amplificador/archivos_kiCad/v2/Ampli_clase_G.sch (KiCad schematic (older format))
At the start: 117 parts, among them J1 Conn_IN, J2 LOAD_CONN, J3 SUPPLY_CONN, J4 CONN_OUT, Q1 BC856, Q10 BC846, Q11 2SC4793, Q14 2SC4793, Q15 2SA1837, Q16 2SC4793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

Commit message: Archivos de KiCad - Correccion de transistor Q7
Parts:
- Q7: value BC856 -> 2SC4793; footprint TO_SOT_Packages_SMD:SOT-23_Handsoldering -> TO_SOT_Packages_THT:TO-220-3_Vertical; symbol BC856 -> Q_NPN_BCE
- Q9: footprint TO_SOT_Packages_THT:TO-126_Vertical -> TO_SOT_Packages_THT:TO-220-3_Vertical
- R37, R40: footprint Resistors_THT:R_Radial_Power_L16.1mm_W9.0mm_P7.37mm -> Resistors_THT:R_Axial_Power_L25.0mm_W9.0mm_P27.94mm
Changed lines of the file:
@@
 F 0 "Q9" H 7700 4625 50  0000 L CNN
 F 1 "2SC4793" H 7700 4550 50  0000 L CNN
-F 2 "TO_SOT_Packages_THT:TO-126_Vertical" H 7700 4475 50  0001 L CIN
+F 2 "TO_SOT_Packages_THT:TO-220-3_Vertical" H 7700 4475 50  0001 L CIN
 F 3 "" H 7500 4550 50  0001 L CNN
 	1    7500 4550
@@
 $EndComp
 $Comp
-L BC856 Q7
+L Q_NPN_BCE Q7
 U 1 1 5D0F592A
 P 7500 1800
 F 0 "Q7" H 7700 1875 50  0000 L CNN
-F 1 "BC856" H 7700 1800 50  0000 L CNN
-F 2 "TO_SOT_Packages_SMD:SOT-23_Handsoldering" H 7700 1725 50  0001 L CIN
+F 1 "2SC4793" H 7700 1800 50  0000 L CNN
+F 2 "TO_SOT_Packages_THT:TO-220-3_Vertical" H 7700 1725 50  0001 L CIN
 F 3 "" H 7500 1800 50  0001 L CNN
 	1    7500 1800
-	1    0    0    1
+	1    0    0    -1
 $EndComp
 $Comp
@@
 F 0 "R40" V 11380 5250 50  0000 C CNN
 F 1 "0.22" V 11300 5250 50  0000 C CNN
-F 2 "Resistors_THT:R_Radial_Power_L16.1mm_W9.0mm_P7.37mm" V 11230 5250 50  0001 C CNN
+F 2 "Resistors_THT:R_Axial_Power_L25.0mm_W9.0mm_P27.94mm" V 11230 5250 50  0001 C CNN
 F 3 "" H 11300 5250 50  0001 C CNN
 	1    11300 5250
@@
 F 0 "R37" V 11380 4500 50  0000 C CNN
 F 1 "0.22" V 11300 4500 50  0000 C CNN
-F 2 "Resistors_THT:R_Radial_Power_L16.1mm_W9.0mm_P7.37mm" V 11230 4500 50  0001 C CNN
+F 2 "Resistors_THT:R_Axial_Power_L25.0mm_W9.0mm_P27.94mm" V 11230 4500 50  0001 C CNN
 F 3 "" H 11300 4500 50  0001 C CNN
 	1    11300 4500
