File: Amplificador/archivos_kiCad/Definitivo/Ampli_clase_G.sch (KiCad schematic (older format))
At the start: 115 parts, among them J1 Conn_IN, J2 LOAD_CONN, J3 SUPPLY_CONN, J4 CONN_OUT, Q1 BC856, Q10 BC846, Q11 2SC4793, Q14 2SC4793, Q15 2SA1837, Q16 2SC4793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

Commit message: Gerbers Files - PCB Amp. terminada
Parts:
- added JP8: Jumper_Feedback, Pin_Headers:Pin_Header_Straight_1x02_Pitch2.54mm, symbol Jumper_NC_Small
- added JP9: Jumper_2ndStage, Pin_Headers:Pin_Header_Straight_1x02_Pitch2.54mm, symbol Jumper_NC_Small
- JP3: value Jumper_NC_Small -> Jumper_Q2
- Q11, Q14, Q15, Q16, Q17, Q9: footprint TO_SOT_Packages_THT:TO-126_Vertical -> TO_SOT_Packages_THT:TO-220-3_Vertical
- Q7: value BC856 -> 2SA1837; footprint TO_SOT_Packages_SMD:SOT-23_Handsoldering -> TO_SOT_Packages_THT:TO-220-3_Vertical; symbol BC856 -> Q_PNP_BCE
- R22: value 390 -> 330
- R3, R4: footprint Resistors_THT:R_Axial_DIN0204_L3.6mm_D1.6mm_P7.62mm_Horizontal -> Resistors_SMD:R_0805_HandSoldering
- R37, R40: footprint Resistors_THT:R_Axial_Power_L20.0mm_W6.4mm_P22.40mm -> Resistors_THT:R_Axial_Power_L25.0mm_W9.0mm_P27.94mm
Connections:
- net GND: now also JP3.2
- net at Q2.1 (B): now also C3.1, R15.2, R16.2; no longer JP3.1
- net at L1.1, Q26.1 (E), Q27.1 (E)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: now also JP8.2; no longer R16.1
- net at C9.1, D6.2 (A), JP6.1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: now also JP9.1
- net at D5.1 (K), JP7.1: now also Q7.2 (C); no longer Q7.3 (C)
- net at R17.1, R18.2: now also Q7.3 (E); no longer Q7.2 (E)
- new net: JP3.1, JP8.1, JP9.2, R16.1
Other:
- moved on the sheet: C8, D1, D2, D3, D4, PR2, R15
