File: Amplificador/construccion/Ampli_clase_G.sch (KiCad schematic (older format))
At the start: 117 parts, among them J1 Conn_IN, J2 LOAD_CONN, J3 SUPPLY_CONN, J4 CONN_OUT, Q1 BC856, Q10 BC846, Q11 2SC4793, Q14 2SC4793, Q15 2SA1837, Q16 2SC4793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

Commit message: cosas
Parts:
- C1: footprint Capacitors_THT:CP_Radial_D4.0mm_P2.00mm -> Capacitors_THT:CP_Radial_D6.3mm_P2.50mm
- C10: footprint Capacitors_THT:CP_Radial_D18.0mm_P7.50mm -> Capacitors_THT:CP_Radial_D22.0mm_P10.00mm_SnapIn
- C12, C4, C5: footprint Capacitors_THT:CP_Radial_D4.0mm_P2.00mm -> Capacitors_THT:CP_Radial_D5.0mm_P2.50mm
- C13: footprint Capacitors_THT:CP_Radial_D16.0mm_P7.50mm -> Capacitors_THT:CP_Radial_D13.0mm_P5.00mm
- C14, C16, C17: footprint Capacitors_THT:CP_Radial_D16.0mm_P7.50mm -> Capacitors_THT:CP_Radial_D14.0mm_P5.00mm
- C3: footprint Capacitors_THT:CP_Radial_D4.0mm_P2.00mm -> Capacitors_THT:CP_Radial_D5.0mm_P2.00mm
- C8: footprint Capacitors_THT:CP_Radial_D10.0mm_P5.00mm -> Capacitors_THT:CP_Radial_D8.0mm_P3.80mm
- Q1, Q2, Q5, Q6: value BC856 -> MMBTA92
- Q10, Q22, Q23, Q24, Q25, Q3, Q4, Q8: value BC846 -> MMBTA42
- Q18, Q19, Q20, Q21: footprint TO_SOT_Packages_THT:TO-220-3_Vertical -> TO_SOT_Packages_THT:TO-264_Vertical
- Q26, Q27: footprint TO_SOT_Packages_THT:TO-92_Molded_Narrow -> TO_SOT_Packages_THT:TO-92_Inline_Wide
- Q7: value 2SC4793 -> 2SA1837; symbol Q_NPN_BCE -> Q_PNP_BCE
- R19: footprint Resistors_THT:R_Axial_DIN0309_L9.0mm_D3.2mm_P12.70mm_Horizontal -> Resistors_THT:R_Axial_DIN0614_L14.3mm_D5.7mm_P15.24mm_Horizontal
- R22: value 390 -> 330
- R37, R40: footprint Resistors_THT:R_Radial_Power_L16.1mm_W9.0mm_P7.37mm -> Resistors_THT:R_Axial_Power_L25.0mm_W9.0mm_P27.94mm
- R39: footprint Resistors_THT:R_Axial_DIN0309_L9.0mm_D3.2mm_P12.70mm_Horizontal -> Resistors_THT:R_Axial_DIN0309_L9.0mm_D3.2mm_P15.24mm_Horizontal
Connections:
- wire segments 242 -> 347

Commit message: Modificacion del esquematico
Cambio de los transistores BC846 y BC856 por MMBTA42 y MMBTA92
Connections:
- wire segments 347 -> 242
